File: pcb/Ghoost Board.kicad_pcb (KiCad board)
At the start: 2 copper layers, 319 x 142.5 mm, 368 parts, among them J1 USB_C_Receptacle_USB2.0_16P, J2 Battery_JST_PH2, SW1 Gateron_Blue, SW10 Gateron_Blue, SW11 Gateron_Blue, SW12 Gateron_Blue, SW13 Gateron_Blue, SW14 Gateron_Blue, SW15 Gateron_Blue, SW16 Gateron_Blue, SW17 Gateron_Blue, SW18 Gateron_Blue, SW19 Gateron_Blue, SW2 Gateron_Blue, SW20 Gateron_Blue, SW21 Gateron_Blue, SW22 Gateron_Blue, SW23 Gateron_Blue, SW24 Gateron_Blue, SW25 Gateron_Blue, SW26 Gateron_Blue, SW27 Gateron_Blue, SW28 Gateron_Blue, SW29 Gateron_Blue, SW3 Gateron_Blue, SW30 Gateron_Blue, SW31 Gateron_Blue, SW32 Gateron_Blue, SW33 Gateron_Blue, SW34 Gateron_Blue, SW35 Gateron_Blue, SW36 Gateron_Blue, SW37 Gateron_Blue, SW38 Gateron_Blue, SW39 Gateron_Blue, SW4 Gateron_Blue, SW40 Gateron_Blue, SW41 Gateron_Blue, SW42 Gateron_Blue, SW43 Gateron_Blue, SW44 Gateron_Blue, SW45 Gateron_Blue, SW46 Gateron_Blue, SW47 Gateron_Blue, SW48 Gateron_Blue, SW49 Gateron_Blue, SW5 Gateron_Blue, SW50 Gateron_Blue, SW51 Gateron_Blue, SW52 Gateron_Blue, SW53 Gateron_Blue, SW54 Gateron_Blue, SW55 Gateron_Blue, SW56 Gateron_Blue, SW57 Gateron_Blue, SW58 Gateron_Blue, SW59 Gateron_Blue, SW6 Gateron_Blue, SW60 Gateron_Blue, SW61 Gateron_Blue, SW62 Gateron_Blue, SW63 Gateron_Blue, SW64 Gateron_Blue, SW65 Gateron_Blue, SW66 Gateron_Blue, SW67 Gateron_Blue, SW68 Gateron_Blue, SW69 Gateron_Blue, SW7 Gateron_Blue, SW70 Gateron_Blue, SW71 Gateron_Blue, SW72 Gateron_Blue, SW73 Gateron_Blue, SW74 Gateron_Blue, SW75 Gateron_Blue, SW76 Gateron_Blue, SW77 Gateron_Blue, SW78 Gateron_Blue, SW79 Gateron_Blue, SW8 Gateron_Blue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

Commit message: yaya
Routing:
- net VBUS: track 2651.5 -> 2639.3 mm
